File: ATTinyAmpDriver.brd (EAGLE design)
At the start: 41.9 x 15.9 mm, 34 parts, among them Q1 SI2301CDS, Q2 BC846, U1 SPX5205M5-L-3-3, U2 ATTINY5-TSHR, U3 MCP6L2-X_SN, X2 INPUT

Commit message: Board Complete
Parts:
- removed X2: INPUT, con-phoenix-254:3POL254
- added U$1: CON_TAILLIGHT, Combined:TAILLIGHT
- moved LED4 7.63 mm to (37.7, 11.1), flipped to the top, turned to 180 degrees
- moved LED2 7.39 mm to (37.5, 5.54), flipped to the bottom, turned to 0 degrees
- moved +5V 7.08 mm to (15.2, 6.48)
- moved C2 7.08 mm to (18.5, 13.4)
- moved R4 7.08 mm to (20.6, 13.4)
- moved R6 7.08 mm to (15.8, 11.4)
- moved RESET 7.08 mm to (20.6, 5.61)
- moved C1 7.08 mm to (13.6, 3.63)
- moved GND 7.08 mm to (12.1, 13.3)
- moved C3 7.08 mm to (16.8, 4.78)
- moved C4 7.08 mm to (23.6, 13.8)
- moved C5 7.08 mm to (23.5, 6.30)
- moved D1 7.08 mm to (13.3, 10.7)
- moved MEASURE 7.08 mm to (17.4, 7.87)
- moved OUTA 7.08 mm to (27.5, 7.16)
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Connections:
- net +14V: now also U$1.H1; no longer X2.1
- net GND: now also U$1.L1, U$1.L2; no longer X2.2
- net N$1: now also U$1.H2; no longer X2.3
Routing:
- net +14V: track 29.2 -> 12.4 mm
- net D-: track 0.00 -> 12.4 mm
- net N$7: track 13.3 -> 4.76 mm, vias 0 -> 1
- net CROSSOVER: track 1.88 -> 9.60 mm, vias 1 -> 0
- net N$3: track 11.2 -> 4.97 mm
- net N$1: track 4.05 -> 10.2 mm, vias 0 -> 1
- net N$10: track 0.00 -> 4.06 mm, vias 0 -> 1
- net GND: vias 4 -> 3
Other:
- board text added: "EWM 20130716 BULB RETROFIT"
- board text removed: "D+"
- board text removed: "D-"
- board text removed: "EWM 20130630 AT DRIVER 3"

Commit message: Fixed pin polarity on Tail Connecter
Connections:
- net +14V: now also U$1.L1; no longer U$1.H1
- net GND: now also U$1.H2; no longer U$1.L1
- net N$1: now also U$1.H1; no longer U$1.H2
Routing:
- net N$1: track 10.2 -> 13.6 mm, vias 1 -> 0
- net +14V: track 12.4 -> 9.79 mm, vias 0 -> 3
- net GND: vias 3 -> 6
- added copper zone on layer 16, net +14V
Changed lines of the file:
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@@
 <vertex x="41.9608" y="4.5212"/>
 <vertex x="41.91" y="0.0254"/>
-<vertex x="30.1244" y="0"/>
-<vertex x="30.1244" y="4.3434"/>
-<vertex x="30.1498" y="5.0546"/>
+<vertex x="30.5054" y="-0.0254"/>
+<vertex x="30.48" y="4.3434"/>
+<vertex x="30.4546" y="5.0546"/>
 <vertex x="28.3972" y="5.0546"/>
 <vertex x="21.1582" y="5.1308"/>
 <vertex x="21.1582" y="2.5146"/>
-<vertex x="10.8712" y="2.5908"/>
-<vertex x="10.8712" y="4.826"/>
-<vertex x="0" y="4.8514"/>
+<vertex x="10.8458" y="2.5908"/>
+<vertex x="10.8458" y="2.286"/>
+<vertex x="-0.0254" y="2.3114"/>
 </polygon>
 <polygon width="0.254" layer="16">
-<vertex x="-0.772" y="16.3422"/>
+<vertex x="-0.3148" y="16.1898"/>
 <vertex x="42.369" y="16.1898"/>
 <vertex x="42.315" y="-0.5784"/>
-<vertex x="-0.726" y="-0.526"/>
+<vertex x="12.2534" y="-0.4752"/>
+<vertex x="12.2682" y="6.4336"/>
+<vertex x="-0.3302" y="6.477"/>
 </polygon>
 <contactref element="GND" pad="P$1"/>
@@
 <via x="24.6634" y="9.9314" extent="1-16" drill="0.6"/>
 <via x="29.6418" y="11.938" extent="1-16" drill="0.6"/>
-<via x="30.4038" y="5.9944" extent="1-16" drill="0.6"/>
+<via x="32.5374" y="5.207" extent="1-16" drill="0.6"/>
 <contactref element="LED1" pad="TH"/>
 <contactref element="LED4" pad="TH"/>
@@
 <contactref element="LED2" pad="TH"/>
 <contactref element="U$1" pad="L2"/>
-<contactref element="U$1" pad="L1"/>
+<contactref element="U$1" pad="H2"/>
+<via x="37.5158" y="8.3058" extent="1-16" drill="0.6"/>
+<via x="2.6162" y="14.605" extent="1-16" drill="0.6"/>
+<via x="2.6924" y="8.2042" extent="1-16" drill="0.6"/>
 </signal>
 <signal name="+14V">
@@
 <contactref element="U1" pad="3"/>
 <polygon width="0.254" layer="1">
-<vertex x="-0.1016" y="3.7084"/>
-<vertex x="10.7188" y="3.556"/>
-<vertex x="10.6934" y="2.1336"/>
+<vertex x="-0.0762" y="1.8288"/>
+<vertex x="12.3444" y="1.8288"/>
+<vertex x="12.319" y="2.159"/>
 <vertex x="21.6662" y="2.0828"/>
 <vertex x="21.6662" y="4.3434"/>
@@
 <vertex x="26.162" y="4.2926"/>
 <vertex x="29.6926" y="4.3434"/>
-<vertex x="26.9748" y="0.0254"/>
+<vertex x="29.718" y="-0.1524"/>
 <vertex x="-0.127" y="-0.1016"/>
 </polygon>
 <contactref element="Q1" pad="P$2"/>
 <contactref element="R2" pad="1"/>
-<contactref element="U$1" pad="H1"/>
-<wire x1="5.334" y1="3.1623" x2="10.6299" y2="3.1623" width="0.6096" layer="1"/>
-<wire x1="10.6299" y1="3.1623" x2="11.43" y2="3.9624" width="0.6096" layer="1"/>
-<wire x1="11.43" y1="3.9624" x2="11.43" y2="4.6482" width="0.6096" layer="1"/>
-<wire x1="11.43" y1="4.6482" x2="12.3698" y2="5.588" width="0.6096" layer="1"/>
-<wire x1="12.3698" y1="7.4676" x2="11.43" y2="7.4676" width="0.6096" layer="1"/>
-<wire x1="11.43" y1="7.4676" x2="11.2268" y2="7.2644" width="0.6096" layer="1"/>
-<wire x1="11.2268" y1="7.2644" x2="11.2268" y2="5.7404" width="0.6096" layer="1"/>
-<wire x1="11.2268" y1="5.7404" x2="11.3792" y2="5.588" width="0.6096" layer="1"/>
-<wire x1="11.3792" y1="5.588" x2="12.3698" y2="5.588" width="0.6096" layer="1"/>
-<wire x1="25.5016" y1="1.6646" x2="29.0392" y2="1.6408" width="0" layer="19" extent="1-1"/>
+<contactref element="U$1" pad="L1"/>
+<polygon width="0.3048" layer="16">
+<vertex x="-0.3302" y="5.9944"/>
+<vertex x="11.5316" y="5.9944"/>
+<vertex x="11.5316" y="-0.2794"/>
+<vertex x="-0.3048" y="-0.2794"/>
+<vertex x="-0.3302" y="3.4798"/>
+</polygon>
+<via x="1.27" y="1.27" extent="1-16" drill="0.6"/>
+<via x="5.3975" y="1.27" extent="1-16" drill="0.6"/>
+<via x="9.525" y="1.27" extent="1-16" drill="0.6"/>
+<wire x1="12.3698" y1="5.588" x2="11.8872" y2="5.588" width="0.4064" layer="1"/>
+<wire x1="11.8872" y1="5.588" x2="11.7348" y2="5.4356" width="0.4064" layer="1"/>
+<wire x1="11.7348" y1="5.4356" x2="11.4808" y2="5.1816" width="0.4064" layer="1"/>
+<wire x1="11.4808" y1="5.1816" x2="11.4808" y2="1.7018" width="0.4064" layer="1"/>
+<wire x1="11.4808" y1="1.7018" x2="11.1252" y2="1.3462" width="0.4064" layer="1"/>
+<wire x1="11.1252" y1="1.3462" x2="9.6012" y2="1.3462" width="0.4064" layer="1"/>
+<wire x1="9.6012" y1="1.3462" x2="9.525" y2="1.27" width="0.4064" layer="1"/>
+<wire x1="12.3698" y1="7.4676" x2="11.7856" y2="7.4676" width="0.4064" layer="1"/>
+<wire x1="11.7856" y1="7.4676" x2="11.176" y2="6.858" width="0.4064" layer="1"/>
+<wire x1="11.176" y1="6.858" x2="11.176" y2="5.9436" width="0.4064" layer="1"/>
+<wire x1="11.176" y1="5.9436" x2="11.7348" y2="5.4356" width="0.4064" layer="1"/>
 </signal>
 <signal name="VCC">
@@
 <signal name="N$1">
 <contactref element="D1" pad="1A"/>
-<contactref element="U$1" pad="H2"/>
-<via x="11.6332" y="12.1412" extent="1-16" drill="0.6" diameter="0.4064" shape="square"/>
-<wire x1="13.3096" y1="9.8434" x2="12.1276" y2="9.8434" width="0.6096" layer="1"/>
-<wire x1="12.1276" y1="9.8434" x2="11.684" y2="10.287" width="0.6096" layer="1"/>
-<wire x1="11.684" y1="10.287" x2="11.684" y2="12.0904" width="0.6096" layer="1"/>
-<wire x1="11.684" y1="12.0904" x2="11.6332" y2="12.1412" width="0.6096" layer="1"/>
-<wire x1="5.334" y1="12.6873" x2="11.0871" y2="12.6873" width="0.6096" layer="16"/>
-<wire x1="11.0871" y1="12.6873" x2="11.6332" y2="12.1412" width="0.6096" layer="16"/>
+<contactref element="U$1" pad="H1"/>
+<wire x1="13.3096" y1="9.8434" x2="11.977" y2="9.8434" width="0.4064" layer="1"/>
+<wire x1="11.977" y1="9.8434" x2="10.287" y2="8.1534" width="0.4064" layer="1"/>
+<wire x1="10.287" y1="8.1534" x2="10.287" y2="3.3528" width="0.4064" layer="1"/>
+<wire x1="10.287" y1="3.3528" x2="10.0584" y2="3.1242" width="0.4064" layer="1"/>
+<wire x1="10.0584" y1="3.1242" x2="5.3721" y2="3.1242" width="0.4064" layer="1"/>
+<wire x1="5.3721" y1="3.1242" x2="5.334" y2="3.1623" width="0.4064" layer="1"/>
 </signal>
 <signal name="N$4">

Commit message: Created programming fixture
Parts:
- +5V, GND, MEASURE, OUTA, PWM, RESET, TPICLK, TPIDATA: device Personal:TPI_PAD -> Combined:TPI_PAD
Changed lines of the file:
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@@
 <grid distance="0.001" unitdist="inch" unit="inch" style="lines" multiple="1" display="no" altdistance="0.025" altunitdist="inch" altunit="inch"/>
 <layers>
-<layer number="1" name="Top" color="4" fill="1" visible="yes" active="yes"/>
-<layer number="16" name="Bottom" color="1" fill="1" visible="yes" active="yes"/>
-<layer number="17" name="Pads" color="2" fill="1" visible="yes" active="yes"/>
-<layer number="18" name="Vias" color="2" fill="1" visible="yes" active="yes"/>
-<layer number="19" name="Unrouted" color="6" fill="1" visible="yes" active="yes"/>
+<layer number="1" name="Top" color="4" fill="1" visible="no" active="yes"/>
+<layer number="16" name="Bottom" color="1" fill="1" visible="no" active="yes"/>
+<layer number="17" name="Pads" color="2" fill="1" visible="no" active="yes"/>
+<layer number="18" name="Vias" color="2" fill="1" visible="no" active="yes"/>
+<layer number="19" name="Unrouted" color="6" fill="1" visible="no" active="yes"/>
 <layer number="20" name="Dimension" color="15" fill="1" visible="yes" active="yes"/>
-<layer number="21" name="tPlace" color="7" fill="1" visible="yes" active="yes"/>
-<layer number="22" name="bPlace" color="7" fill="1" visible="yes" active="yes"/>
-<layer number="23" name="tOrigins" color="15" fill="1" visible="yes" active="yes"/>
-<layer number="24" name="bOrigins" color="15" fill="1" visible="yes" active="yes"/>
+<layer number="21" name="tPlace" color="7" fill="1" visible="no" active="yes"/>
+<layer number="22" name="bPlace" color="7" fill="1" visible="no" active="yes"/>
+<layer number="23" name="tOrigins" color="15" fill="1" visible="no" active="yes"/>
+<layer number="24" name="bOrigins" color="15" fill="1" visible="no" active="yes"/>
 <layer number="25" name="tNames" color="7" fill="1" visible="yes" active="yes"/>
-<layer number="26" name="bNames" color="7" fill="1" visible="yes" active="yes"/>
+<layer number="26" name="bNames" color="7" fill="1" visible="no" active="yes"/>
 <layer number="27" name="tValues" color="7" fill="1" visible="no" active="yes"/>
 <layer number="28" name="bValues" color="7" fill="1" visible="no" active="yes"/>
@@
 <layer number="37" name="tTest" color="7" fill="1" visible="no" active="yes"/>
 <layer number="38" name="bTest" color="7" fill="1" visible="no" active="yes"/>
-<layer number="39" name="tKeepout" color="4" fill="11" visible="yes" active="yes"/>
-<layer number="40" name="bKeepout" color="1" fill="11" visible="yes" active="yes"/>
-<layer number="41" name="tRestrict" color="4" fill="10" visible="yes" active="yes"/>
-<layer number="42" name="bRestrict" color="1" fill="10" visible="yes" active="yes"/>
-<layer number="43" name="vRestrict" color="2" fill="10" visible="yes" active="yes"/>
+<layer number="39" name="tKeepout" color="4" fill="11" visible="no" active="yes"/>
+<layer number="40" name="bKeepout" color="1" fill="11" visible="no" active="yes"/>
+<layer number="41" name="tRestrict" color="4" fill="10" visible="no" active="yes"/>
+<layer number="42" name="bRestrict" color="1" fill="10" visible="no" active="yes"/>
+<layer number="43" name="vRestrict" color="2" fill="10" visible="no" active="yes"/>
 <layer number="44" name="Drills" color="7" fill="1" visible="no" active="yes"/>
-<layer number="45" name="Holes" color="7" fill="1" visible="yes" active="yes"/>
+<layer number="45" name="Holes" color="7" fill="1" visible="no" active="yes"/>
 <layer number="46" name="Milling" color="3" fill="1" visible="no" active="yes"/>
-<layer number="47" name="Measures" color="7" fill="1" visible="yes" active="yes"/>
+<layer number="47" name="Measures" color="7" fill="1" visible="no" active="yes"/>
 <layer number="48" name="Document" color="7" fill="1" visible="no" active="yes"/>
 <layer number="49" name="Reference" color="7" fill="1" visible="no" active="yes"/>
-<layer number="51" name="tDocu" color="7" fill="1" visible="yes" active="yes"/>
-<layer number="52" name="bDocu" color="7" fill="1" visible="yes" active="yes"/>
+<layer number="51" name="tDocu" color="7" fill="1" visible="no" active="yes"/>
+<layer number="52" name="bDocu" color="7" fill="1" visible="no" active="yes"/>
 <layer number="91" name="Nets" color="2" fill="1" visible="no" active="no"/>
 <layer number="92" name="Busses" color="1" fill="1" visible="no" active="no"/>
@@
 <layer number="97" name="Info" color="7" fill="1" visible="no" active="no"/>
 <layer number="98" name="Guide" color="6" fill="1" visible="no" active="no"/>
+<layer number="100" name="TestPads" color="7" fill="1" visible="yes" active="yes"/>
 <layer number="250" name="Descript" color="3" fill="1" visible="no" active="no"/>
 <layer number="251" name="SMDround" color="12" fill="11" visible="no" active="no"/>
@@
 <text x="15.3416" y="7.4168" size="0.8128" layer="25">V</text>
 <text x="16.1036" y="7.4168" size="0.8128" layer="25">M</text>
+<dimension x1="0" y1="0" x2="41.91" y2="0" x3="20.955" y3="-4.7498" textsize="1.778" layer="20" unit="inch" precision="3"/>
+<dimension x1="0" y1="15.875" x2="0" y2="0" x3="-2.8194" y3="7.9375" textsize="1.778" layer="20" unit="inch" precision="3"/>
 </plain>
 <attributes>
@@
 <attribute name="DIGIKEY_COST" value=".04" x="25.5016" y="2.5146" size="1.778" layer="27" rot="R90" display="off"/>
 </element>
-<element name="TPIDATA" library="Personal" package="TPI_PAD" value="TPI" x="20.5994" y="4.0132"/>
-<element name="TPICLK" library="Personal" package="TPI_PAD" value="TPI" x="16.6878" y="13.0302"/>
-<element name="+5V" library="Personal" package="TPI_PAD" value="TPI" x="15.2146" y="6.477"/>
-<element name="GND" library="Personal" package="TPI_PAD" value="TPI" x="12.0904" y="13.2842"/>
+<element name="TPIDATA" library="Combined" package="TPI_PAD" value="TPI" x="20.5994" y="4.0132"/>
+<element name="TPICLK" library="Combined" package="TPI_PAD" value="TPI" x="16.6878" y="13.0302"/>
+<element name="+5V" library="Combined" package="TPI_PAD" value="TPI" x="15.2146" y="6.477"/>
+<element name="GND" library="Combined" package="TPI_PAD" value="TPI" x="12.0904" y="13.2842"/>
 <element name="C1" library="resistor" package="C0603" value="10n" x="13.589" y="3.6322" smashed="yes" rot="R180">
 <attribute name="NAME" x="13.97" y="2.3368" size="0.8128" layer="25" rot="R180"/>
@@
 <attribute name="DIGIKEY_COST" value=".10" x="13.589" y="3.6322" size="1.778" layer="27" rot="R180" display="off"/>
 </element>
-<element name="RESET" library="Personal" package="TPI_PAD" value="TPI" x="20.6248" y="5.6134"/>
+<element name="RESET" library="Combined" package="TPI_PAD" value="TPI" x="20.6248" y="5.6134"/>
 <element name="R9" library="resistor" package="R0603" value="28.7K" x="29.591" y="8.5344" smashed="yes" rot="R90">
 <attribute name="DIGIKEY" value="RMCF0603FT28R7CT-ND" x="29.591" y="8.5344" size="1.778" layer="27" rot="R90" display="off"/>
@@
 <attribute name="VALUE" x="29.6418" y="9.4234" size="1.27" layer="27" rot="R270"/>
 </element>
-<element name="PWM" library="Personal" package="TPI_PAD" value="TPI" x="29.1084" y="4.8006"/>
-<element name="MEASURE" library="Personal" package="TPI_PAD" value="TPI" x="17.4498" y="7.874"/>
-<element name="OUTA" library="Personal" package="TPI_PAD" value="TPI" x="27.4828" y="7.1628"/>
+<element name="PWM" library="Combined" package="TPI_PAD" value="TPI" x="29.1084" y="4.8006"/>
+<element name="MEASURE" library="Combined" package="TPI_PAD" value="TPI" x="17.4498" y="7.874"/>
+<element name="OUTA" library="Combined" package="TPI_PAD" value="TPI" x="27.4828" y="7.1628"/>
 <element name="LED1" library="Combined" package="CREE_XP-E" value="LUXEON_REBELCREE_XP-E" x="37.5412" y="2.8194"/>
 <element name="LED2" library="Combined" package="CREE_XP-E" value="LUXEON_REBELCREE_XP-E" x="37.5412" y="5.5372" rot="MR0"/>
@@
 </signal>
 </signals>
-<errors>
-</errors>
 </board>
 </drawing>
